Commit message: updates after stretch

File: charger_description/urdf/charger.urdf.xacro (robot description, xacro)
@@ -1,6 +1,5 @@
 <?xml version="1.0"?>
 <robot xmlns:xacro="http://wiki.ros.org/xacro" name="robot">
-  <!-- helper macro -->
-  <xacro:include filename="$(find charger_description)/urdf/inc/create_link.xacro"/>
+ <xacro:include filename="$(find charger_description)/urdf/inc/create_link.xacro"/>
   <xacro:create_link
       link_name="base"
@@ -31,22 +30,19 @@
       mesh_name="tag"
   />
-  <!-- joints - main serial chain -->
-  <joint name="joint_1" type="fixed">
+  <!-- helper macro -->
+  <joint name="bar_joint" type="fixed">
+    <origin rpy="0.00000 0.00000 0.00000" xyz="-0.01821 +0.00135 -0.70465"/>
     <parent link="bar"/>
     <child link="base"/>
-    <origin xyz="-0.026013 0 -0.235144" rpy="0 0 0"/>
-    <axis xyz="0 0 1"/>
   </joint>
-  <joint name="joint_2" type="fixed">
+  <joint name="port_joint" type="fixed">
+    <origin rpy="0.00000 0.00000 0.00000" xyz="0.06053 0.01121 -0.58665"/>
     <parent link="bar"/>
     <child link="port"/>
-    <origin xyz="0.068162 0 0.053566" rpy="0 0 0"/>
-    <axis xyz="0 0 1"/>
   </joint>
-  <joint name="joint_3" type="fixed">
+  <joint name="tag_joint" type="fixed">
+    <origin rpy="0.00000 0.00000 0.00000" xyz="-0.06575 0.00037 -0.38023"/>
     <parent link="tag_203"/>
     <child link="bar"/>
-    <origin xyz="-0.013006 0 -0.257653" rpy="0 0 0"/>
-    <axis xyz="0 0 1"/>
   </joint>
 </robot>

Commit message: workign version before localiza and goign back to docking after reminders

File: charger_description/urdf/charger.urdf.xacro (robot description, xacro)
@@ -1,12 +1,6 @@
 <?xml version="1.0"?>
 <robot xmlns:xacro="http://wiki.ros.org/xacro" name="robot">
- <xacro:include filename="$(find charger_description)/urdf/inc/create_link.xacro"/>
-  <xacro:create_link
-      link_name="base"
-      xyz_offset="0 0 0"
-      rpy_offset="0 0 0"
-      mesh_package="charger_description"
-      mesh_name="base"
-  />
+  <!-- helper macro -->
+  <xacro:include filename="$(find charger_description)/urdf/inc/create_link.xacro"/>
   <xacro:create_link
       link_name="bar"
@@ -30,19 +24,16 @@
       mesh_name="tag"
   />
-  <!-- helper macro -->
-  <joint name="bar_joint" type="fixed">
-    <origin rpy="0.00000 0.00000 0.00000" xyz="-0.01821 +0.00135 -0.70465"/>
-    <parent link="bar"/>
-    <child link="base"/>
-  </joint>
-  <joint name="port_joint" type="fixed">
-    <origin rpy="0.00000 0.00000 0.00000" xyz="0.06053 0.01121 -0.58665"/>
+  <!-- joints - main serial chain -->
+  <joint name="joint_1" type="fixed">
     <parent link="bar"/>
     <child link="port"/>
+    <origin xyz="0.068162 0 0.053566" rpy="0 0 0"/>
+    <axis xyz="0 0 1"/>
   </joint>
-  <joint name="tag_joint" type="fixed">
-    <origin rpy="0.00000 0.00000 0.00000" xyz="-0.06575 0.00037 -0.38023"/>
+  <joint name="joint_2" type="fixed">
     <parent link="tag_203"/>
     <child link="bar"/>
+    <origin xyz="-0.013006 0 -0.257653" rpy="0 0 0"/>
+    <axis xyz="0 0 1"/>
   </joint>
 </robot>

Commit message: Calibrate new docking syestem transforms
*Reverse the charging port

*Change docking camera transform for new camera mount

Decreased tag to bar length to lower the tag height

File: charger_description/urdf/charger.urdf.xacro (robot description, xacro)
@@ -34,5 +34,5 @@
     <parent link="tag_203"/>
     <child link="bar"/>
-    <origin xyz="-0.013006 0 -0.257653" rpy="0 0 0"/>
+    <origin xyz="-0.013006 0 -0.177" rpy="0 0 0"/>
     <axis xyz="0 0 1"/>
   </joint>
